File: hardware/sinodude-rp2354/sinodude-rp2354.kicad_pcb (KiCad board)
At the start: 2 copper layers, 64 x 36 mm, 93 parts, among them J1 USB-C, J2 SWD TC2030-IDC latching, J4 DUT, Q1 2N7002, SW1 BOOTSEL, SW2 RESET, U1 RP2354A, U2 AMS1117-3.3, U3 TPS2114APW, U4 SN74LVC8T245PW, U5 SN74LVC1T45DBV, U6 SN74LVC1T45DBV, Y1 12MHz/CL10pF/ESR50R/ABM8-272-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

Commit message: hardware: strengthen the data-line pull-ups for protoB and SWD
SinoLink runs four wire protocols over this header: protoA JTAG
bit-bang, protoB single-wire pulse-width, CMSIS-DAP SWD, and Andes
AICE. All four are carried here already, now that TDA works: the three
lines that reverse sit on their own translator with a GPIO DIR, and the
four that never reverse share U4.

The one thing that did not carry over was pull-up strength. SinoLink
translates its data wire with a PCA9306, a passive pass-FET that cannot
drive high, so its 1k on the MCU side and switched 330R on the target
side are its high-side driver rather than a bus bias. The SN74LVC1T45
here is push-pull and drives high on its own, so no switched pull-up is
wanted; what is left is the released line, where the target drives
open-drain and the resistor alone sets the rising edge.

R31 and R33 go 10k to 1k, matching SinoLink's static value: about 30 ns
into the ~30 pF a short ribbon presents, against ~300 ns at 10k, which
matters where the protocol is decoded by measuring pulse widths. R29 on
nRST stays 10k, since a reset line is not clocked.

Also corrects F1's stated margin. U3's limit is not a flat 333 mA:
scaling the datasheet's 700 ohm row to R15 = 750 ohm gives
280 / 336 / 467 mA, so the worst case through F1 is ~540 mA, not the
400-430 mA claimed. Still inside the 750 mA hold.
Parts:
- R31, R33: value 10k -> 1k
Changed lines of the file:
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@@
 			)
 		)
-		(property "Value" "10k"
+		(property "Value" "1k"
 			(at 0 -1.43 180)
 			(unlocked yes)
@@
 			)
 		)
-		(property "LCSC" "C25804"
+		(property "LCSC" "C21190"
 			(at 0 0 180)
 			(layer "B.Fab")
@@
 			)
 		)
-		(property "Value" "10k"
+		(property "Value" "1k"
 			(at 0 -1.43 180)
 			(unlocked yes)
@@
 			)
 		)
-		(property "LCSC" "C25804"
-			(at 0 0 180)
-			(layer "B.Fab")
+		(property "LCSC" "C21190"
+			(at 0 0 180)
+			(layer "B.Fab")

Commit message: hardware: label the DUT header pins on the bottom silk
The IDC body covers the top silk around J4, so there was nowhere to
read the pinout from. The bottom had no J4 silk at all.

Adds a pinout legend on B.Silkscreen in the clear 11 x 11 mm area just
above the header, laid out to match the connector, plus a pin-1 dot in
the gap between R23/R24 and the header. Odd pins sit at the lower board
x and so does the odd column of the legend, so the two mirror together
and the legend still reads correctly from underneath.

Per-pin labels beside each pad do not fit: the strip west of the odd
column is 1.56 mm and the east side is taken by the D4-D9 clamp column.
Other:
- board text added: "1 VTGT"
- board text added: "10 GND"
- board text added: "2 TCK"
- board text added: "3 GND"
- board text added: "4 TDI"
- board text added: "5 GND"
- board text added: "6 TMS"
- board text added: "7 TDA"
- board text added: "8 TDO"
- board text added: "9 nRST"
- board text added: "J4 DUT"
Changed lines of the file:
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@@
 		)
+	)
+	(gr_circle
+		(center 167.7 99.92)
+		(end 168.05 99.92)
+		(stroke
+			(width 0.15)
+			(type default)
+		)
+		(fill yes)
+		(layer "B.SilkS")
 	)
 	(gr_arc
@@
 		(layer "Edge.Cuts")
 	)
+	(gr_text "1 VTGT"
+		(at 164.6 91.3 0)
+		(layer "B.SilkS")
+		(effects
+			(font
+				(size 0.8 0.8)
+				(thickness 0.15)
+			)
+			(justify mirror)
+		)
+	)
+	(gr_text "3 GND"
+		(at 164.6 93 0)
+		(layer "B.SilkS")
+		(effects
+			(font
+				(size 0.8 0.8)
+				(thickness 0.15)
+			)
+			(justify mirror)
+		)
+	)
+	(gr_text "5 GND"
+		(at 164.6 94.7 0)
+		(layer "B.SilkS")
+		(effects
+			(font
+				(size 0.8 0.8)
+				(thickness 0.15)
+			)
+			(justify mirror)
+		)
+	)
+	(gr_text "7 TDA"
+		(at 164.6 96.4 0)
+		(layer "B.SilkS")
+		(effects
+			(font
+				(size 0.8 0.8)
+				(thickness 0.15)
+			)
+			(justify mirror)
+		)
+	)
+	(gr_text "9 nRST"
+		(at 164.6 98.1 0)
+		(layer "B.SilkS")
+		(effects
+			(font
+				(size 0.8 0.8)
+				(thickness 0.15)
+			)
+			(justify mirror)
+		)
+	)
+	(gr_text "J4 DUT"
+		(at 167.5 89.4 0)
+		(layer "B.SilkS")
+		(effects
+			(font
+				(size 0.8 0.8)
+				(thickness 0.15)
+			)
+			(justify mirror)
+		)
+	)
+	(gr_text "2 TCK"
+		(at 170.4 91.3 0)
+		(layer "B.SilkS")
+		(effects
+			(font
+				(size 0.8 0.8)
+				(thickness 0.15)
+			)
+			(justify mirror)
+		)
+	)
+	(gr_text "4 TDI"
+		(at 170.4 93 0)
+		(layer "B.SilkS")
+		(effects
+			(font
+				(size 0.8 0.8)
+				(thickness 0.15)
+			)
+			(justify mirror)
+		)
+	)
+	(gr_text "6 TMS"
+		(at 170.4 94.7 0)
+		(layer "B.SilkS")
+		(effects
+			(font
+				(size 0.8 0.8)
+				(thickness 0.15)
+			)
+			(justify mirror)
+		)
+	)
+	(gr_text "8 TDO"
+		(at 170.4 96.4 0)
+		(layer "B.SilkS")
+		(effects
+			(font
+				(size 0.8 0.8)
+				(thickness 0.15)
+			)
+			(justify mirror)
+		)
+	)
+	(gr_text "10 GND"
+		(at 170.4 98.1 0)
+		(layer "B.SilkS")
+		(effects
+			(font
+				(size 0.8 0.8)
+				(thickness 0.15)
+			)
+			(justify mirror)
+		)
+	)
 	(segment
